File: picoprobe-pcb/picoprobe-pcb.kicad_pcb (KiCad board)
At the start: 2 copper layers, 2 parts, among them J1 Conn_01x06_Pin, U1 Pico

Commit message: First draft
What:

Why:

How:

Tags:
Parts:
- U1: footprint RPi_Pico:RPi_Pico_SMD_TH -> MCU_RaspberryPi_and_Boards:RPi_Pico_SMD_TH
- moved U1 44.9 mm to (151.1, 90.2)
- moved J1 37.2 mm to (144.8, 121.9)
Connections:
- J1 pad 4: unconnected-(J1-Pin_4-Pad4) -> Net-(J1-Pin_4)
- J1 pad 5: unconnected-(J1-Pin_5-Pad5) -> Net-(J1-Pin_5)
- J1 pad 6: unconnected-(J1-Pin_6-Pad6) -> Net-(J1-Pin_6)
- U1 pad 38: unconnected-(U1-GND-Pad38) -> Net-(J1-Pin_6)
- U1 pad 39: unconnected-(U1-VSYS-Pad39) -> Net-(J1-Pin_5)
- U1 pad 4: unconnected-(U1-GPIO2-Pad4) -> Net-(J1-Pin_4)
- U1 pad 41: Net-(J1-Pin_1) -> unconnected-(U1-SWCLK-Pad41)
- U1 pad 42: Net-(J1-Pin_2) -> unconnected-(U1-GND-Pad42)
- U1 pad 43: Net-(J1-Pin_3) -> unconnected-(U1-SWDIO-Pad43)
- U1 pad 5: unconnected-(U1-GPIO3-Pad5) -> Net-(J1-Pin_3)
- U1 pad 6: unconnected-(U1-GPIO4-Pad6) -> Net-(J1-Pin_2)
- U1 pad 7: unconnected-(U1-GPIO5-Pad7) -> Net-(J1-Pin_1)
Routing:
- net Net-(J1-Pin_6): track 0.00 -> 58.3 mm
- net Net-(J1-Pin_4): track 0.00 -> 55.9 mm
- net Net-(J1-Pin_5): track 0.00 -> 55.4 mm
- net Net-(J1-Pin_3): track 0.00 -> 48.9 mm
- net Net-(J1-Pin_1): track 0.00 -> 48.5 mm
- net Net-(J1-Pin_2): track 0.00 -> 47.1 mm
